File: hardware/schematics/stonyman_breakout.sch (KiCad schematic (older format))
At the start: 1 part

Commit message: updated schematic
Other:
- note added: "P12:13"
- note added: "P12:14"
- note added: "P12:17"
- note added: "P12:18"
- note added: "P12:19"
- note added: "P12:20"
- note added: "P12:7"
- note added: "P12:9"
- note removed: "P10:13"
- note removed: "P10:14"
- note removed: "P10:17"
- note removed: "P10:18"
- note removed: "P10:19"
- note removed: "P10:20"
- note removed: "P10:7"
- note removed: "P10:9"
Changed lines of the file:
@@
 $EndComp
 Text Notes 8400 1500 0    60   ~ 0
-P10:7
+P12:7
 Text Notes 8400 1850 0    60   ~ 0
-P10:9
+P12:9
 Text Notes 6100 4650 0    60   ~ 0
 6, CS
@@
 Connection ~ 3750 3650
 Text Notes 8400 2150 0    60   ~ 0
-P10:13
+P12:13
 Text Notes 8400 2450 0    60   ~ 0
-P10:14
+P12:14
 Text Notes 8400 2750 0    60   ~ 0
-P10:17
+P12:17
 Text Notes 8400 3050 0    60   ~ 0
-P10:18
+P12:18
 Text Notes 8400 3350 0    60   ~ 0
-P10:19
+P12:19
 Text Notes 8400 3650 0    60   ~ 0
-P10:20
+P12:20
 Text Notes 8400 4100 0    60   Italic 12
 SmartFusion\nBoard

Commit message: updated to work on 3.3 V stonyman
Parts:
- 20K: symbol R -> R-RESCUE-stonyman_breakout
Other:
- note added: "GND, 2"
- note removed: "GND"
Changed lines of the file:
@@
 EESchema Schematic File Version 2
+LIBS:stonyman_breakout-rescue
 LIBS:power
 LIBS:device
@@
 LIBS:memory
 LIBS:xilinx
-LIBS:special
 LIBS:microcontrollers
 LIBS:dsp
@@
 LIBS:contrib
 LIBS:valves
+LIBS:stonyman_breakout-cache
 EELAYER 25 0
 EELAYER END
@@
 Va, 1
 Text Notes 5600 5650 0    60   ~ 0
-GND
+GND, 2
 $Comp
 L +5V #PWR?
@@
 	8350 3050 8350 3000
 $Comp
-L R 20K
+L R-RESCUE-stonyman_breakout 20K
 U 1 1 55109811
 P 3750 3900

Commit message: updated schematic
Parts:
- added C1: 1 uF, symbol CP
- renumbered 20K to 30K
Connections:
- net +5V: now also C1.1
- net GNDREF: now also C1.2
Changed lines of the file:
@@
 	8350 3050 8350 3000
 $Comp
-L R-RESCUE-stonyman_breakout 20K
+L R-RESCUE-stonyman_breakout 30K
 U 1 1 55109811
 P 3750 3900
-F 0 "20K" V 3830 3900 50  0000 C CNN
+F 0 "30K" V 3830 3900 50  0000 C CIB
 F 1 "R" V 3757 3901 50  0000 C CNN
 F 2 "" V 3680 3900 30  0000 C CNN
@@
 Text Notes 8500 4350 0    60   ~ 0
 P10:3
+$Comp
+L +5V #PWR?
+U 1 1 56AF7983
+P 2550 5150
+F 0 "#PWR?" H 2550 5000 50  0001 C CNN
+F 1 "+5V" H 2550 5290 50  0000 C CNN
+F 2 "" H 2550 5150 60  0000 C CNN
+F 3 "" H 2550 5150 60  0000 C CNN
+	1    2550 5150
+	1    0    0    -1
+$EndComp
+$Comp
+L GNDREF #PWR?
+U 1 1 56AF799A
+P 2550 5550
+F 0 "#PWR?" H 2550 5300 50  0001 C CNN
+F 1 "GNDREF" H 2550 5400 50  0000 C CNN
+F 2 "" H 2550 5550 60  0000 C CNN
+F 3 "" H 2550 5550 60  0000 C CNN
+	1    2550 5550
+	1    0    0    -1
+$EndComp
+$Comp
+L CP C1
+U 1 1 56AF79B0
+P 2550 5300
+F 0 "C1" H 2575 5400 50  0000 L CNN
+F 1 "1 uF" H 2575 5200 50  0000 L CNN
+F 2 "" H 2588 5150 30  0000 C CNN
+F 3 "" H 2550 5300 60  0000 C CNN
+	1    2550 5300
+	1    0    0    -1
+$EndComp
+Wire Wire Line
+	2550 5450 2550 5550
 $EndSCHEMATC
