File: hardware/senseye-2_temple/rev_a/senseye-2_temple.brd (EAGLE design)
At the start: 142.2 x 88.3 mm, 2 parts, among them J1 M11X2, U1 FH19SC-22S-0.5SH(05)

Commit message: routed and marked holes
Parts:
- moved J1 59.1 mm to (-32.1, -9.53)
- moved U1 22.9 mm to (-11.7, -7.62), turned to 90 degrees
Connections:
- net SDATA renamed SCLK0
- removed net N$12: J1.21
- removed net N$21: J1.20
- removed net N$22: J1.22
- removed net N$38: U1.3
- removed net N$39: U1.2
- removed net N$40: U1.1
- removed net SCLK: J1.18, U1.5
- new net SCLK1: J1.20, U1.3
- new net SDATA0: J1.16, U1.7
- new net SDATA1: J1.19, U1.4
- net CS1: now also J1.18, U1.5; no longer J1.16, U1.7
- net GND: now also J1.21, U1.2
- net LED: now also J1.22, U1.1; no longer J1.19, U1.4
Routing:
- net RESP0: track 0.00 -> 35.9 mm
- net RESV0: track 0.00 -> 33.0 mm
- net INCP0: track 0.00 -> 31.0 mm
- net INPHI0: track 0.00 -> 29.4 mm, vias 0 -> 1
- net INCV0: track 0.00 -> 28.2 mm
- net RESP1: track 0.00 -> 27.0 mm, vias 0 -> 1
- net OUTENABLE0: track 0.00 -> 25.8 mm
- net RESV1: track 0.00 -> 24.8 mm, vias 0 -> 1
- net INCP1: track 0.00 -> 23.4 mm
- net INPHI1: track 0.00 -> 22.4 mm, vias 0 -> 1
- net INCV1: track 0.00 -> 21.0 mm
- net CS0: track 0.00 -> 19.9 mm, vias 0 -> 1
- net OUTENABLE1: track 0.00 -> 18.6 mm
- net SCLK0: track 0.00 -> 17.5 mm, vias 0 -> 1
- net SDATA0: track 0.00 -> 16.2 mm
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- added copper zone on layer 1, net GND
- added copper zone on layer 16, net VCC
Other:
- board size 142.2 x 88.3 mm -> 142.5 x 43.2 mm
- board text added: "CS0"
- board text added: "CS1"
- board text added: "GND"
- board text added: "IP0"
- board text added: "IP1"
- board text added: "IPH0"
- board text added: "IPH1"
- board text added: "IV0"
- board text added: "IV1"
- board text added: "LED"
- board text added: "OE0"
- board text added: "OE1"
- board text added: "RP0"
- board text added: "RP1"
- board text added: "RV0"
- board text added: "RV1"
- board text added: "SC0"
- board text added: "SC1"
- board text added: "SD0"
- board text added: "SD1"
- board text added: "VCC"
