File: hardware/senseye-2_temple/rev_a/senseye-2_temple.sch (EAGLE design)
At the start: 2 parts, among them J1 M11X2, U1 FH19SC-22S-0.5SH(05)

Commit message: routed and marked holes
Connections:
- net SDATA renamed SCLK0
- removed net N$12: J1.21
- removed net N$21: J1.20
- removed net N$22: J1.22
- removed net N$38: U1.3
- removed net N$39: U1.2
- removed net N$40: U1.1
- removed net SCLK: J1.18, U1.5
- new net SCLK1: J1.20, U1.3
- new net SDATA0: J1.16, U1.7
- new net SDATA1: J1.19, U1.4
- net CS1: now also J1.18, U1.5; no longer J1.16, U1.7
- net GND: now also J1.21, U1.2
- net LED: now also J1.22, U1.1; no longer J1.19, U1.4
