File: hardware/senseye-2_temple_r/rev_a/senseye-2_temple_r.brd (EAGLE design)
At the start: 142.5 x 43.2 mm, 2 parts, among them J1 M11X2, U1 FH19SC-22S-0.5SH(05)

Commit message: moved all to 0,0 origin
Parts:
- moved J1 77.3 mm to (32.1, 33.7), flipped to the bottom
- moved U1 49.2 mm to (11.7, 35.6), flipped to the bottom
Routing:
- added copper zone on layer 16, net GND
- added copper zone on layer 1, net VCC
- removed copper zone on layer 1, net GND
- removed copper zone on layer 16, net VCC
Other:
- outline, holes or cut-outs redrawn
