File: hardware/eagle/senseye-2/rev_a/senseye-2.brd (EAGLE design)
At the start: 149.8 x 55.3 mm, 19 parts, among them U1 ADC121S101, U2 ADC121S101, U3 ADC121S101

Commit message: updated eagle with 30k resistor
Parts:
- R3, R4, R5: value 10k -> 30k
Changed lines of the file:
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@@
 <?xml version="1.0" encoding="utf-8"?>
 <!DOCTYPE eagle SYSTEM "eagle.dtd">
-<eagle version="6.5.0">
+<eagle version="7.5.0">
 <drawing>
 <settings>
@@
 <pass name="Default">
 <param name="RoutingGrid" value="50mil"/>
+<param name="AutoGrid" value="1"/>
+<param name="Efforts" value="0"/>
+<param name="TopRouterVariant" value="1"/>
 <param name="tpViaShape" value="round"/>
 <param name="PrefDir.1" value="|"/>
@@
 </element>
 <element name="JP3" library="senseye" package="1X09" value="STONYMAN" x="23.8125" y="50.4825" smashed="yes"/>
-<element name="R3" library="passives" package="0402_RES" value="10k" x="62.23" y="46.99" smashed="yes" rot="MR90">
+<element name="R3" library="passives" package="0402_RES" value="30k" x="62.23" y="46.99" smashed="yes" rot="MR90">
 <attribute name="NAME" x="61.595" y="46.0375" size="1.27" layer="26" font="vector" ratio="10" rot="MR180" align="bottom-center"/>
 </element>
 <element name="JP5" library="senseye" package="FH19SC-22S-0.5SH(05)" value="FH19SC-22S-0.5SH(05)" x="139.955" y="34.735" rot="MR270"/>
-<element name="R4" library="passives" package="0402_RES" value="10k" x="23.495" y="5.08" smashed="yes" rot="MR90">
+<element name="R4" library="passives" package="0402_RES" value="30k" x="23.495" y="5.08" smashed="yes" rot="MR90">
 <attribute name="NAME" x="24.765" y="5.7785" size="1.27" layer="26" font="vector" ratio="10" rot="MR0" align="bottom-center"/>
 </element>
@@
 <attribute name="NAME" x="16.8275" y="51.435" size="1.27" layer="26" font="vector" ratio="10" rot="MR0"/>
 </element>
-<element name="R5" library="passives" package="0402_RES" value="10k" x="19.685" y="49.2125" smashed="yes" rot="MR90">
+<element name="R5" library="passives" package="0402_RES" value="30k" x="19.685" y="49.2125" smashed="yes" rot="MR90">
 <attribute name="NAME" x="19.685" y="50.2285" size="1.27" layer="26" font="vector" ratio="10" rot="MR0" align="bottom-center"/>
 </element>
